File: Hardware/ESP32_DRONE_WAAR.kicad_sch (KiCad schematic)
At the start: 0 parts

Commit message: Version 2 11/13 15:26
Parts:
- added DWM1: DWM3000, RF_Module:DWM1000, symbol RF_Module:DWM3000
- added HS1: Heatsink_Pad, symbol Mechanical:Heatsink_Pad
- added J1: USB_B_Micro, symbol Connector:USB_B_Micro
- added U1: CP2104, Package_DFN_QFN:QFN-24-1EP_4x4mm_P0.5mm_EP2.6x2.6mm, symbol Interface_USB:CP2104
- added U2: ESP32-S2-WROVER, RF_Module:ESP32-S2-WROVER, symbol RF_Module:ESP32-S2-WROVER
Connections:
- new net: U1.2 (GND), U1.25 (GND)
- new net: J1.3 (D+), U1.3 (D+)
- new net: J1.2 (D-), U1.4 (D-)
- new net: J1.1 (VBUS), U1.8 (VBUS)
- new net: DWM1.16 (VSS), DWM1.21 (VSS), DWM1.23 (VSS), DWM1.24 (VSS), DWM1.8 (VSS)
- new net: U2.1 (GND), U2.26 (GND), U2.42 (GND), U2.43 (GND)
- new net GND: HS1.1, J1.5 (GND), J1.6 (Shield)

Commit message: v2 11/16/25 18:27
Parts:
- added C1, C11, C2, C3, C4, C6, C8, C9: 10µF, symbol Device:C
- added C10, C7: 100nF, symbol Device:C
- added C12: 0.1µF, symbol Device:C
- added C5: 1.0µF, symbol Device:C
- added D1: 1N4005, Diode_THT:D_DO-41_SOD81_P10.16mm_Horizontal, symbol Diode:1N4005
- added D2, D3, D4, D5, D6: LED, symbol Device:LED
- added J2, J3: Conn_01x04_MountingPin, symbol Connector_Generic_MountingPin:Conn_01x04_MountingPin
- added Q1, Q2: S8050, Package_TO_SOT_THT:TO-92_Inline, symbol Transistor_BJT:S8050
- added R1, R11, R4, R5: 10k, symbol Device:R_US
- added R10, R6, R7, R8, R9: 1k, symbol Device:R_US
- added R12, R13, R14, R15: 470R, symbol Device:R_US
- added R2, R3: 470, symbol Device:R_US
- added SW1, SW2: SW_MEC_5G, symbol Switch:SW_MEC_5G
- added U3: LD1117V33, Package_TO_SOT_THT:TO-220-3_Vertical, symbol Regulator_Linear:LD1117V33
- added U4: ME6217C33M5G, 0my_project:SOT-23-5L, symbol dd:ME6217C33M5G
Connections:
- net GND: now also DWM1.16 (VSS), DWM1.21 (VSS), DWM1.23 (VSS), DWM1.24 (VSS), DWM1.8 (VSS), U1.2 (GND), U1.25 (GND), U2.1 (GND), U2.26 (GND), U2.42 (GND), U2.43 (GND), C1.1, C10.2, C11.2, C12.1, C2.2, C3.2, C4.2, C5.2, C6.2, C7.2, C8.2, C9.2, D3.1 (K), D4.1 (K), D5.1 (K), D6.1 (K), J2.2 (Pin_2), J2.MP (MountPin), J3.2 (Pin_2), J3.4 (Pin_4), J3.MP (MountPin), R11.2, R3.2, SW1.1 (A), SW1.2 (A), SW2.1 (A), SW2.2 (A), U3.1 (GND), U4.2 (Vss)
- net at U1.16 (VPP): now also C9.1
- net RTS: now reaches U1.19 (~{RTS})
- net RTS: now also Q2.1 (E), R6.1
- net RXD: now reaches U1.20 (RXD)
- net RXD: now also J2.3 (Pin_3)
- net TXD: now reaches U1.21 (TXD)
- net TXD: now also J2.4 (Pin_4)
- net DTR: now reaches U1.23 (~{DTR})
- net DTR: now also Q1.1 (E), R7.1
- net +3V3: now reaches U1.5 (VIO)
- net +3V3: now also DWM1.5 (VDDAON), DWM1.6 (VDD3V3), DWM1.7 (VDD3V3), U1.6 (VDD), U1.7 (REGIN), U2.2 (3V3), C1.2, C11.1, C12.2, C5.1, C8.1, D2.2 (A), J3.1 (Pin_1), R4.1, R5.1, U4.5 (Vout)
- net VBUS: now reaches J1.1 (VBUS), U1.8 (VBUS)
- net VBUS: now also C4.1, C6.1, C7.1, D1.2 (A), R1.1, U4.1 (Vin)
- net at DWM1.1 (EXTON): now also R8.2
- net GPIO5: now reaches DWM1.10 (GPIO5/EXTTXE/SPIPOL)
- net GPIO4: now reaches DWM1.11 (GPIO4/EXTPA)
- net LEDTX: now reaches DWM1.12 (GPIO3/TXLED)
- net LEDTX: now also R12.1
- net LEDRX: now reaches DWM1.13 (GPIO2/RXLED)
- net LEDRX: now also R13.1
- net LEDSFD: now reaches DWM1.14 (GPIO1/SFDLED)
- net LEDSFD: now also R14.1
- net LEDRXOK: now reaches DWM1.15 (GPIO0/RXOKLED)
- net LEDRXOK: now also R15.1
- net IO4: now reaches DWM1.17 (~{SPICS})
- net IO23: now reaches DWM1.18 (SPIMOSI)
- net at DWM1.19 (SPIMISO): no longer names the net of DWM1.19 (SPIMISO)
- net at DWM1.2 (WAKEUP): now also R9.2
- net IO18: now reaches DWM1.20 (SPICLK)
- net IO34: now reaches DWM1.22 (IRQ/GPIO8)
- net IO34: now also R11.1
- net at DWM1.3 (~{RST}): now also R10.1
- net GPIO6: now reaches DWM1.9 (GPIO6/EXTRXE/SPIHA)
- net RESET: now reaches U2.41 (EN)
- net RESET: now also J3.3 (Pin_3), Q2.3 (C), SW1.3 (B), SW1.4 (B)
- new net: D5.2 (A), R14.2
- new net: D2.1 (K), R3.1
- new net: D3.2 (A), R12.2
- new net: D6.2 (A), R15.2
- new net: D4.2 (A), R13.2
- new net: Q1.2 (B), R6.2
- new net: Q2.2 (B), R7.2
- new net: R2.2, SW2.3 (B), SW2.4 (B)
- new net: C10.1, R4.2
- new net: C3.1, U3.2 (VO)
- new net CLOCK: R1.2, U4.3 (CE)
- new net IO0: Q1.3 (C), R2.1, R5.2
- new net IO27: R10.2
- new net IO32: R9.1
- new net IO33: R8.1
- new net VDDV5: C2.1, D1.1 (K), J2.1 (Pin_1), U3.3 (VI)
- no-connect marks 0 -> 15
Other:
- moved on the sheet: DWM1, HS1, U2
