File: Hardware/ESP32_DRONE_WAAR.kicad_sch (KiCad schematic)
At the start: 0 parts

Commit message: Add files via upload
Parts:
- added C1, C11, C2, C3, C4, C6, C8, C9: 10µF, symbol Device:C
- added C10, C7: 100nF, symbol Device:C
- added C12: 0.1µF, symbol Device:C
- added C13: 0.01uf, symbol Device:C_Small_US
- added C14: 0.1uf, symbol Device:C_Small_US
- added C15, C18: 0.1uF, symbol Device:C_Small_US
- added C16: 4.7uF, symbol Device:C_Small_US
- added C17: 10uF, symbol Device:C_Small_US
- added C5: 1.0µF, symbol Device:C
- added D1: 1N4005, Diode_THT:D_DO-41_SOD81_P10.16mm_Horizontal, symbol Diode:1N4005
- added D2, D3, D4, D5, D6: LED, symbol Device:LED
- added DWM1: DWM3000, RF_Module:DWM1000, symbol RF_Module:DWM3000
- added HS1: Heatsink_Pad, symbol Mechanical:Heatsink_Pad
- added J1: USB_B_Micro, symbol Connector:USB_B_Micro
- added J2, J3: Conn_01x04_MountingPin, symbol Connector_Generic_MountingPin:Conn_01x04_MountingPin
- added Q1, Q2: S8050, Package_TO_SOT_THT:TO-92_Inline, symbol Transistor_BJT:S8050
- added R1, R11, R16, R17, R18, R19, R20, R21, R22, R4, R5: 10k, symbol Device:R_US
- added R10, R6, R7, R8, R9: 1k, symbol Device:R_US
- added R12, R13, R14, R15: 470R, symbol Device:R_US
- added R2, R3: 470, symbol Device:R_US
- added SW1, SW2, SW3: SW_MEC_5G, symbol Switch:SW_MEC_5G
- added U1: CP2104, Package_DFN_QFN:QFN-24-1EP_4x4mm_P0.5mm_EP2.6x2.6mm, symbol Interface_USB:CP2104
- added U2: ESP32-S2-WROVER, RF_Module:ESP32-S2-WROVER, symbol RF_Module:ESP32-S2-WROVER
- added U3: LD1117V33, Package_TO_SOT_THT:TO-220-3_Vertical, symbol Regulator_Linear:LD1117V33
- added U4: ME6217C33M5G, 0my_project:SOT-23-5L, symbol dd:ME6217C33M5G
- added U5: MPU-9250, Sensor_Motion:InvenSense_QFN-24_3x3mm_P0.4mm, symbol Sensor_Motion:MPU-9250
- added U6: LT1962-3.3V LDO, Package_SO:MSOP-8_3x3mm_P0.65mm, symbol Regulator_Linear:LT1962-3.3
Connections:
- new net: D5.2 (A), R14.2
- new net: R16.2, U5.24 (SDA/MOSI)
- new net: C9.1, U1.16 (VPP)
- new net: J1.3 (D+), U1.3 (D+)
- new net: J1.2 (D-), U1.4 (D-)
- new net: D2.1 (K), R3.1
- new net: C15.1, U5.10 (REGOUT)
- new net: R18.1, U5.11 (FSYNC)
- new net: R21.1, U5.21 (AUX_DA)
- new net: R20.1, U5.22 (~{CS})
- new net: R17.1, U5.23 (SCL/SCLK)
- new net: R22.1, U5.7 (AUX_CL)
- new net: R19.1, U5.9 (AD0/MISO)
- new net: D3.2 (A), R12.2
- new net: D6.2 (A), R15.2
- new net: D4.2 (A), R13.2
- new net: DWM1.1 (EXTON), R8.2
- new net: DWM1.2 (WAKEUP), R9.2
- new net: DWM1.3 (~{RST}), R10.1
- new net: Q1.2 (B), R6.2
- new net: Q2.2 (B), R7.2
- new net: R2.2, SW2.3 (B), SW2.4 (B)
- new net: C10.1, R4.2
- new net: C3.1, U3.2 (VO)
- new net +3.3V: C17.1, C18.1, SW3.3 (B), SW3.4 (B), U6.1 (OUT)
- new net +3V3: C1.2, C11.1, C12.2, C13.1, C14.1, C5.1, C8.1, D2.2 (A), DWM1.5 (VDDAON), DWM1.6 (VDD3V3), DWM1.7 (VDD3V3), J3.1 (Pin_1), R16.1, R17.2, R20.2, R21.2, R22.2, R4.1, R5.1, U1.5 (VIO), U1.6 (VDD), U1.7 (REGIN), U2.2 (3V3), U4.5 (Vout), U5.1 (RESV_VDDIO), U5.13 (VDD), U5.8 (VDDIO)
- new net +5V: C16.1, SW3.1 (A), SW3.2 (A), U6.5 (~{SHDN}), U6.8 (IN)
- new net CLOCK: R1.2, U4.3 (CE)
- new net DTR: Q1.1 (E), R7.1, U1.23 (~{DTR})
- new net GND: C1.1, C10.2, C11.2, C12.1, C13.2, C14.2, C15.2, C16.2, C17.2, C18.2, C2.2, C3.2, C4.2, C5.2, C6.2, C7.2, C8.2, C9.2, D3.1 (K), D4.1 (K), D5.1 (K), D6.1 (K), DWM1.16 (VSS), DWM1.21 (VSS), DWM1.23 (VSS), DWM1.24 (VSS), DWM1.8 (VSS), HS1.1, J1.5 (GND), J1.6 (Shield), J2.2 (Pin_2), J2.MP (MountPin), J3.2 (Pin_2), J3.4 (Pin_4), J3.MP (MountPin), R11.2, R18.2, R19.2, R3.2, SW1.1 (A), SW1.2 (A), SW2.1 (A), SW2.2 (A), U1.2 (GND), U1.25 (GND), U2.1 (GND), U2.26 (GND), U2.42 (GND), U2.43 (GND), U3.1 (GND), U4.2 (Vss), U5.18 (GND), U5.20 (RESV_GND), U6.4 (GND)
- new net GPIO4: DWM1.11 (GPIO4/EXTPA)
- new net GPIO5: DWM1.10 (GPIO5/EXTTXE/SPIPOL)
- new net GPIO6: DWM1.9 (GPIO6/EXTRXE/SPIHA)
- new net IO0: Q1.3 (C), R2.1, R5.2
- new net IO18: DWM1.20 (SPICLK)
- new net IO23: DWM1.18 (SPIMOSI)
- new net IO27: R10.2
- new net IO32: R9.1
- new net IO33: R8.1
- new net IO34: DWM1.22 (IRQ/GPIO8), R11.1
- new net IO4: DWM1.17 (~{SPICS})
- new net LEDRX: DWM1.13 (GPIO2/RXLED), R13.1
- new net LEDRXOK: DWM1.15 (GPIO0/RXOKLED), R15.1
- new net LEDSFD: DWM1.14 (GPIO1/SFDLED), R14.1
- new net LEDTX: DWM1.12 (GPIO3/TXLED), R12.1
- new net RESET: J3.3 (Pin_3), Q2.3 (C), SW1.3 (B), SW1.4 (B), U2.41 (EN)
- new net RTS: Q2.1 (E), R6.1, U1.19 (~{RTS})
- new net RXD: J2.3 (Pin_3), U1.20 (RXD)
- new net TXD: J2.4 (Pin_4), U1.21 (TXD)
- new net VBUS: C4.1, C6.1, C7.1, D1.2 (A), J1.1 (VBUS), R1.1, U1.8 (VBUS), U4.1 (Vin)
- new net VDDV5: C2.1, D1.1 (K), J2.1 (Pin_1), U3.3 (VI)
- no-connect marks 0 -> 15

Commit message: Add files via upload
Parts:
- removed U2: ESP32-S2-WROVER, RF_Module:ESP32-S2-WROVER, symbol RF_Module:ESP32-S2-WROVER
- added C19: 0.1 uF, symbol Device:C_Small_US
- added C20: 1 uF, symbol Device:C_Small_US
- added U7: BME280, Sensors:PSON65P250X250X100-8N, symbol Sensor:BME280
- added U8: ESP32-WROOM-32, RF_Module:ESP32-WROOM-32, symbol RF_Module:ESP32-WROOM-32
Connections:
- net +3V3: now also C19.1, C20.1, U7.2 (CSB), U7.3 (SDI), U7.4 (SCK), U7.6 (VDDIO), U7.8 (VDD), U8.2 (VDD), U8.27 (IO16)
- net GND: now also C19.2, C20.2, U7.1 (GND), U7.7 (GND), U8.1 (GND), U8.15 (GND), U8.38 (GND), U8.39 (GND)
- net SDA_IMU: now reaches R16.2, U5.24 (SDA/MOSI)
- net SCL_IMU: now reaches R17.1, U5.23 (SCL/SCLK)
- new net SCL_BME: U8.28 (IO17)
- no-connect marks 15 -> 17
Other:
- note added: "RESET"
- moved on the sheet: C13, C14, C15, C16, C17, C18, D1, J3, R16, R17, R18, R19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
